File: PIR-ESP-V10.brd (EAGLE design)
At the start: 54.3 x 67.3 mm, 13 parts

Commit message: add wires
Parts:
- removed D4: (no value), SparkFun-LED:LED5MM
- removed U$1: ESP-12-E, esp8266modules:ESP-12-E
- added C2: 4.7u, SparkFun-Passives:1206
- added C3, C4: 0.1u, SparkFun-Passives:1206
- added Q1, Q2: 200mA/50V, SparkFun-DiscreteSemi:SOT23-3
- added R1, R2, R3, R4, R5: (no value), SparkFun-Passives:1206
- added RST/PRG: SWITCH, SparkFun-Electromechanical:TACTILE-PTH-SIDEEZ
- added U$2: ESP-12, esp8266modules:ESP-12
- MENU: value SWITCH-MOMENTARY-2SIDE_EZ -> SWITCH
- moved PIR 45.1 mm to (38.1, 7.62), turned to 270 degrees
- moved SG1 43.3 mm to (10.2, 15.2)
- moved FTDI 32.1 mm to (38.1, 34.3), turned to 90 degrees
- moved PANIC 31.4 mm to (38.1, 12.7), turned to 90 degrees
- moved C1 10.2 mm to (27.9, 14.0)
- moved 3V3 6.48 mm to (21.6, 14.0)
- moved JP3 6.35 mm to (21.6, 2.54)
- moved MENU 5.08 mm to (10.2, 2.54)
- moved D1 1.27 mm to (11.4, 25.4), turned to 270 degrees
- turned D2 to 270 degrees
- turned D3 to 270 degrees
Connections:
- new net 3V3: 3V3.2, 3V3.4, C1.1, R5.1, U$2.CH_PD, U$2.VCC
- new net 5V: 3V3.3, C2.1, JP3.VBUS, PIR.1
- new net GPIO0: Q2.3, U$2.GPIO0
- new net N$1: D1.A, U$2.GPIO12
- new net N$10: D2.A, U$2.GPIO13
- new net N$11: D3.A, U$2.GPIO14
- new net N$12: PIR.3, U$2.GPIO2
- new net N$14: C4.2, Q2.1, R4.1
- new net N$16: Q1.3, R4.2, R5.2
- new net N$5: FTDI.2, U$2.RX
- new net N$6: D1.K, R1.2
- new net N$7: D2.K, R2.2
- new net N$8: D3.K, R3.2
- new net N$9: PANIC.2, U$2.GPIO4
- new net RST/PRG: C3.2, Q1.1, RST/PRG.2, U$2.RESET
- net GND: now also C1.2, C2.2, C3.1, C4.1, FTDI.6, JP3.GND, JP3.MT1, JP3.MT2, MENU.2, PANIC.1, PIR.2, Q1.2, Q2.2, R1.1, R2.1, R3.1, RST/PRG.1, SG1.-, U$2.GND, U$2.GPIO15
- net N$2: now also SG1.+, U$2.GPIO5; no longer 3V3.4
- net N$3: now also FTDI.3, U$2.TX; no longer 3V3.2, C1.1
- net N$4: now also MENU.1, U$2.GPIO16; no longer 3V3.3
Other:
- board size 54.3 x 67.3 mm -> 43.2 x 50.8 mm
